Commit message: Blad w pythonie (lab3)

File: lab2/urdf/my_robot.urdf (robot description, URDF)
Before this commit: robot firstRobot, 4 links, 3 joints
Links:
- link l1: geometry visual box size=${l_width} ${params['i1']['l_len']} ${l_width}
- link l2: geometry visual box size=${l_width} ${params['i2']['l_len']} ${l_width}
- link l3: geometry visual box size=${l_width} ${l_width} ${params['i3']['l_len']}
Joints:
- joint base_l1: origin xyz=${params['i1']['j_xyz']} rpy=${params['i1']['j_rpy']} -> xyz=${params['i1']['j_xyz']} rpy=${params['i2']['j_rpy']}
- joint l1_l2: origin xyz=${params['i2']['j_xyz']} rpy=${params['i2']['j_rpy']} -> xyz=${params['i2']['j_xyz']} rpy=${params['i3']['j_rpy']}
- joint l2_l3: origin xyz=${params['i3']['j_xyz']} rpy=${params['i3']['j_rpy']} -> xyz=${params['i3']['j_xyz']} rpy=0 0 0

File: lab2/urdf/my_robot_movable.urdf (robot description, URDF)
Before this commit: robot firstRobot, 4 links, 3 joints
Links:
- link l1: geometry visual box size=${l_width} ${params['i1']['l_len']} ${l_width}
- link l2: geometry visual box size=${l_width} ${params['i2']['l_len']} ${l_width}
- link l3: geometry visual box size=${l_width} ${params['i3']['l_len']} ${l_width}
Joints:
- joint base_l1: origin xyz=${params['i1']['j_xyz']} rpy=${params['i1']['j_rpy']} -> xyz=${params['i1']['j_xyz']} rpy=${params['i2']['j_rpy']}
- joint l1_l2: origin xyz=${params['i2']['j_xyz']} rpy=${params['i2']['j_rpy']} -> xyz=${params['i2']['j_xyz']} rpy=${params['i3']['j_rpy']}
- joint l2_l3: axis 0 0 1 -> 0 1 0
