Commit message: Przesuniecie strzalki

File: lab2/urdfPrimo/my_robot.urdf (robot description, URDF)
Before this commit: robot firstRobot, 4 links, 3 joints
Links:
- link l3: geometry visual box size=${l_width} ${l_width} ${params['i3']['l_len']}
Joints:
- joint base_l1: axis 0 1 0 -> 0 0 1; limit lower=${params['i1']['slide']} upper=0 effort=1000.0 velocity=0.5 -> (none); origin xyz=0 0 0 rpy=${params['i2']['j_rpy']} -> xyz=${params['i1']['j_xyz']} rpy=${params['i2']['j_rpy']}; type prismatic -> fixed
- joint l1_l2: axis 0 1 0 -> 0 0 1; limit lower=${params['i2']['slide']} upper=0 effort=1000.0 velocity=0.5 -> (none); type prismatic -> fixed
- joint l2_l3: axis 0 1 0 -> 0 0 1; limit lower=${params['i3']['slide']} upper=0 effort=1000.0 velocity=0.5 -> (none); origin xyz=${params['i3']['j_xyz']} rpy=${params['i3']['j_rpy']} -> xyz=${params['i3']['j_xyz']} rpy=0 0 0; type prismatic -> fixed

File: lab2/urdfPrimo/my_robot_movable.urdf (robot description, URDF)
Before this commit: robot firstRobot, 4 links, 3 joints
Joints:
- joint base_l1: origin xyz=0 0 0 rpy=${params['i2']['j_rpy']} -> xyz=${params['i1']['j_xyz']} rpy=${params['i2']['j_rpy']}
